Commit message: dsfasdfasdf

File: src/catbot_control/urdf/catbot.urdf.xacro (robot description, xacro)
@@ -4,18 +4,10 @@
   <xacro:include filename="$(find catbot_description)/robot.urdf" />
   <ros2_control name="ODrives" type="system">
-    <xacro:unless value="${use_mock_hardware}">
-      <hardware>
-        <plugin>odrive_ros2_control_plugin/ODriveHardwareInterface</plugin>
-        <param name="can">can0</param>
-      </hardware>
-    </xacro:unless>
-    <xacro:if value="${use_mock_hardware}">
-      <hardware>
-        <plugin>mock_components/GenericSystem</plugin>
-        <param name="calculate_dynamics">true</param>
-      </hardware>
-    </xacro:if>
+    <hardware>
+      <plugin>odrive_ros2_control_plugin/ODriveHardwareInterface</plugin>
+      <param name="can">can0</param>
+    </hardware>
     <joint name="FL_hip">
-      <param name="node_id">0</param>
+      <param name="node_id">4</param>
       <command_interface name="position" />
       <state_interface name="position" />
@@ -30,6 +22,6 @@
       <state_interface name="effort" />
     </joint>
-    <joint name="FL_b">
-      <param name="node_id">2</param>
+    <joint name="FL_l">
+      <param name="node_id">9</param>
       <command_interface name="position" />
       <state_interface name="position" />
@@ -38,5 +30,5 @@
     </joint>
     <joint name="FR_hip">
-      <param name="node_id">3</param>
+      <param name="node_id">10</param>
       <command_interface name="position" />
       <state_interface name="position" />
@@ -45,5 +37,5 @@
     </joint>
     <joint name="FR_a">
-      <param name="node_id">4</param>
+      <param name="node_id">6</param>
       <command_interface name="position" />
       <state_interface name="position" />
@@ -51,6 +43,6 @@
       <state_interface name="effort" />
     </joint>
-    <joint name="FR_b">
-      <param name="node_id">5</param>
+    <joint name="FR_l">
+      <param name="node_id">11</param>
       <command_interface name="position" />
       <state_interface name="position" />
@@ -59,5 +51,5 @@
     </joint>
     <joint name="BL_hip">
-      <param name="node_id">6</param>
+      <param name="node_id">5</param>
       <command_interface name="position" />
       <state_interface name="position" />
@@ -72,5 +64,5 @@
       <state_interface name="effort" />
     </joint>
-    <joint name="BL_b">
+    <joint name="BL_l">
       <param name="node_id">8</param>
       <command_interface name="position" />
@@ -80,5 +72,5 @@
     </joint>
     <joint name="BR_hip">
-      <param name="node_id">9</param>
+      <param name="node_id">12</param>
       <command_interface name="position" />
       <state_interface name="position" />
@@ -87,5 +79,5 @@
     </joint>
     <joint name="BR_a">
-      <param name="node_id">10</param>
+      <param name="node_id">3</param>
       <command_interface name="position" />
       <state_interface name="position" />
@@ -93,6 +85,6 @@
       <state_interface name="effort" />
     </joint>
-    <joint name="BR_b">
-      <param name="node_id">11</param>
+    <joint name="BR_l">
+      <param name="node_id">2</param>
       <command_interface name="position" />
       <state_interface name="position" />
@@ -101,3 +93,24 @@
     </joint>
   </ros2_control>
+  <!-- <ros2_control name="IMU" type="sensor">
+    <hardware>
+      <plugin>icm20948_hardware/ICM20948Interface</plugin>
+      <param name="i2c_device">/dev/i2c-7</param>
+      <param name="i2c_address">105</param>
+      <param name="reverse_accel">[true, false, false]</param>
+      <param name="reverse_gyro">[false, true, true]</param>
+    </hardware>
+    <sensor name="imu">
+      <state_interface name="orientation.x" />
+      <state_interface name="orientation.y" />
+      <state_interface name="orientation.z" />
+      <state_interface name="orientation.w" />
+      <state_interface name="angular_velocity.x" />
+      <state_interface name="angular_velocity.y" />
+      <state_interface name="angular_velocity.z" />
+      <state_interface name="linear_acceleration.x" />
+      <state_interface name="linear_acceleration.y" />
+      <state_interface name="linear_acceleration.z" />
+    </sensor>
+  </ros2_control> -->
 </robot>
